File: 0.1/base/ferris.kicad_pcb (KiCad board)
At the start: 2 copper layers, 225 x 95.2 mm, 99 parts, among them J1 USB C, K0_0 KEYSW, K0_1 KEYSW, K0_2 KEYSW, K0_3 KEYSW, K0_4 KEYSW, K0_5 KEYSW, K0_6 KEYSW, K0_7 KEYSW, K0_8 KEYSW, K0_9 KEYSW, K1_0 KEYSW, K1_1 KEYSW, K1_2 KEYSW, K1_3 KEYSW, K1_4 KEYSW, K1_5 KEYSW, K1_6 KEYSW, K1_7 KEYSW, K1_8 KEYSW, K1_9 KEYSW, K2_0 KEYSW, K2_1 KEYSW, K2_2 KEYSW, K2_3 KEYSW, K2_4 KEYSW, K2_5 KEYSW, K2_6 KEYSW, K2_7 KEYSW, K2_8 KEYSW, K2_9 KEYSW, K3_3 KEYSW, K3_4 KEYSW, K3_5 KEYSW, K3_6 KEYSW, SW1 Reset, U1 ATmega32U4-AU, U2 MCP23017_SO, Y1 Crystal

Commit message: Use ferris_pcb_art in 0.1/base
Parts:
- removed the G*** at (188.0, 83.0)
- G***: footprint ferris:mask -> copper_pads:ferris
- G***: footprint ferris:safe_rust -> silkscreens:safe_rust
- G***: footprint ferris:unsafe_rust -> silkscreens:unsafe_rust

Commit message: 0.1/base: update footprints from schematic
Parts:
- C1, C2: value 22pF -> 22p
- C10, C3, C4, C5, C6, C9: value 0.1uF -> 0.1u
- C7: value 4.7uF -> 4.7u
- C8: value 1uF -> 1u
- K0_0, K0_1, K0_2, K0_3, K0_4, K0_5, K0_6, K0_7, K0_8, K0_9, K1_0, K1_1, K1_2, K1_3, K1_4, K1_5, K1_6, K1_7, K1_8, K1_9, K2_0, K2_1, K2_2, K2_3, K2_4, K2_5, K2_6, K2_7, K2_8, K2_9, K3_3, K3_4, K3_5, K3_6: footprint ferris:SW_PG1350 -> switches:Choc_PG1350_MX_Spacing
- R1, R2, R9: value 10kΩ -> 10k
- R3, R4: value 22Ω -> 22
- R5, R6: value 5.1KΩ -> 5.1K
- R7, R8: value 4.7kΩ -> 4.7k
- SW1: value Reset -> SW_PUSH
