File: 0.1/base/ferris.sch (KiCad schematic (older format))
At the start: 95 parts, among them J1 USB C, K0_0 KEYSW, K0_1 KEYSW, K0_2 KEYSW, K0_3 KEYSW, K0_4 KEYSW, K0_5 KEYSW, K0_6 KEYSW, K0_7 KEYSW, K0_8 KEYSW, K0_9 KEYSW, K1_0 KEYSW, K1_1 KEYSW, K1_2 KEYSW, K1_3 KEYSW, K1_4 KEYSW, K1_5 KEYSW, K1_6 KEYSW, K1_7 KEYSW, K1_8 KEYSW, K1_9 KEYSW, K2_0 KEYSW, K2_1 KEYSW, K2_2 KEYSW, K2_3 KEYSW, K2_4 KEYSW, K2_5 KEYSW, K2_6 KEYSW, K2_7 KEYSW, K2_8 KEYSW, K2_9 KEYSW, K3_3 KEYSW, K3_4 KEYSW, K3_5 KEYSW, K3_6 KEYSW, SW1 SW_PUSH, U1 ATmega32U4-AU, U2 MCP23017_SO, Y1 Crystal

Commit message: Update switch footprints
Parts:
- K0_0, K0_1, K0_2, K0_3, K0_4, K0_5, K0_6, K0_7, K0_8, K0_9, K1_0, K1_1, K1_2, K1_3, K1_4, K1_5, K1_6, K1_7, K1_8, K1_9, K2_0, K2_1, K2_2, K2_3, K2_4, K2_5, K2_6, K2_7, K2_8, K2_9, K3_3, K3_4, K3_5, K3_6: footprint ferris:SW_PG1350 -> switches:Choc_PG1350_MX_Spacing
Changed lines of the file:
@@
 F 0 "K0_0" H 1350 1433 60  0000 C CNN
 F 1 "KEYSW" H 1350 1100 60  0001 C CNN
-F 2 "ferris:SW_PG1350" H 1350 1200 60  0001 C CNN
+F 2 "switches:Choc_PG1350_MX_Spacing" H 1350 1200 60  0001 C CNN
 F 3 "" H 1350 1200 60  0000 C CNN
 F 4 "C489144" H 1350 1200 50  0001 C CNN "LCSC Part #"
@@
 F 0 "K1_0" H 1350 2033 60  0000 C CNN
 F 1 "KEYSW" H 1350 1700 60  0001 C CNN
-F 2 "ferris:SW_PG1350" H 1350 1800 60  0001 C CNN
+F 2 "switches:Choc_PG1350_MX_Spacing" H 1350 1800 60  0001 C CNN
 F 3 "" H 1350 1800 60  0000 C CNN
 	1    1350 1800
@@
 F 0 "K1_1" H 2050 2033 60  0000 C CNN
 F 1 "KEYSW" H 2050 1700 60  0001 C CNN
-F 2 "ferris:SW_PG1350" H 2050 1800 60  0001 C CNN
+F 2 "switches:Choc_PG1350_MX_Spacing" H 2050 1800 60  0001 C CNN
 F 3 "" H 2050 1800 60  0000 C CNN
 	1    2050 1800
@@
 F 0 "K0_2" H 2750 1433 60  0000 C CNN
 F 1 "KEYSW" H 2750 1100 60  0001 C CNN
-F 2 "ferris:SW_PG1350" H 2750 1200 60  0001 C CNN
+F 2 "switches:Choc_PG1350_MX_Spacing" H 2750 1200 60  0001 C CNN
 F 3 "" H 2750 1200 60  0000 C CNN
 	1    2750 1200
@@
 F 0 "K0_1" H 2050 1433 60  0000 C CNN
 F 1 "KEYSW" H 2050 1100 60  0001 C CNN
-F 2 "ferris:SW_PG1350" H 2050 1200 60  0001 C CNN
+F 2 "switches:Choc_PG1350_MX_Spacing" H 2050 1200 60  0001 C CNN
 F 3 "" H 2050 1200 60  0000 C CNN
 	1    2050 1200
@@
 F 0 "K1_2" H 2750 2033 60  0000 C CNN
 F 1 "KEYSW" H 2750 1700 60  0001 C CNN
-F 2 "ferris:SW_PG1350" H 2750 1800 60  0001 C CNN
+F 2 "switches:Choc_PG1350_MX_Spacing" H 2750 1800 60  0001 C CNN
 F 3 "" H 2750 1800 60  0000 C CNN
 	1    2750 1800
@@
 F 0 "K2_0" H 1350 2633 60  0000 C CNN
 F 1 "KEYSW" H 1350 2300 60  0001 C CNN
-F 2 "ferris:SW_PG1350" H 1350 2400 60  0001 C CNN
+F 2 "switches:Choc_PG1350_MX_Spacing" H 1350 2400 60  0001 C CNN
 F 3 "" H 1350 2400 60  0000 C CNN
 	1    1350 2400
@@
 F 0 "K2_1" H 2050 2633 60  0000 C CNN
 F 1 "KEYSW" H 2050 2300 60  0001 C CNN
-F 2 "ferris:SW_PG1350" H 2050 2400 60  0001 C CNN
+F 2 "switches:Choc_PG1350_MX_Spacing" H 2050 2400 60  0001 C CNN
 F 3 "" H 2050 2400 60  0000 C CNN
 	1    2050 2400
@@
 F 0 "K2_2" H 2750 2633 60  0000 C CNN
 F 1 "KEYSW" H 2750 2300 60  0001 C CNN
-F 2 "ferris:SW_PG1350" H 2750 2400 60  0001 C CNN
+F 2 "switches:Choc_PG1350_MX_Spacing" H 2750 2400 60  0001 C CNN
 F 3 "" H 2750 2400 60  0000 C CNN
 	1    2750 2400
@@
 F 0 "K0_3" H 3450 1433 60  0000 C CNN
 F 1 "KEYSW" H 3450 1100 60  0001 C CNN
-F 2 "ferris:SW_PG1350" H 3450 1200 60  0001 C CNN
+F 2 "switches:Choc_PG1350_MX_Spacing" H 3450 1200 60  0001 C CNN
 F 3 "" H 3450 1200 60  0000 C CNN
 	1    3450 1200
@@
 F 0 "K1_3" H 3450 2033 60  0000 C CNN
 F 1 "KEYSW" H 3450 1700 60  0001 C CNN
-F 2 "ferris:SW_PG1350" H 3450 1800 60  0001 C CNN
+F 2 "switches:Choc_PG1350_MX_Spacing" H 3450 1800 60  0001 C CNN
 F 3 "" H 3450 1800 60  0000 C CNN
 	1    3450 1800
@@
 F 0 "K2_3" H 3450 2633 60  0000 C CNN
 F 1 "KEYSW" H 3450 2300 60  0001 C CNN
-F 2 "ferris:SW_PG1350" H 3450 2400 60  0001 C CNN
+F 2 "switches:Choc_PG1350_MX_Spacing" H 3450 2400 60  0001 C CNN
 F 3 "" H 3450 2400 60  0000 C CNN
 	1    3450 2400
@@
 F 0 "K0_4" H 4150 1433 60  0000 C CNN
 F 1 "KEYSW" H 4150 1100 60  0001 C CNN
-F 2 "ferris:SW_PG1350" H 4150 1200 60  0001 C CNN
+F 2 "switches:Choc_PG1350_MX_Spacing" H 4150 1200 60  0001 C CNN
 F 3 "" H 4150 1200 60  0000 C CNN
 	1    4150 1200
@@
 F 0 "K1_4" H 4150 2033 60  0000 C CNN
 F 1 "KEYSW" H 4150 1700 60  0001 C CNN
-F 2 "ferris:SW_PG1350" H 4150 1800 60  0001 C CNN
+F 2 "switches:Choc_PG1350_MX_Spacing" H 4150 1800 60  0001 C CNN
 F 3 "" H 4150 1800 60  0000 C CNN
 	1    4150 1800
@@
 F 0 "K2_4" H 4150 2633 60  0000 C CNN
 F 1 "KEYSW" H 4150 2300 60  0001 C CNN
-F 2 "ferris:SW_PG1350" H 4150 2400 60  0001 C CNN
+F 2 "switches:Choc_PG1350_MX_Spacing" H 4150 2400 60  0001 C CNN
 F 3 "" H 4150 2400 60  0000 C CNN
 	1    4150 2400
@@
 F 0 "K3_3" H 3450 3233 60  0000 C CNN
 F 1 "KEYSW" H 3450 2900 60  0001 C CNN
-F 2 "ferris:SW_PG1350" H 3450 3000 60  0001 C CNN
+F 2 "switches:Choc_PG1350_MX_Spacing" H 3450 3000 60  0001 C CNN
 F 3 "" H 3450 3000 60  0000 C CNN
 	1    3450 3000
@@
 F 0 "K3_4" H 4150 3233 60  0000 C CNN
 F 1 "KEYSW" H 4150 2900 60  0001 C CNN
-F 2 "ferris:SW_PG1350" H 4150 3000 60  0001 C CNN
+F 2 "switches:Choc_PG1350_MX_Spacing" H 4150 3000 60  0001 C CNN
 F 3 "" H 4150 3000 60  0000 C CNN
 	1    4150 3000
@@
 F 0 "K0_5" H 7450 1433 60  0000 C CNN
 F 1 "KEYSW" H 7450 1100 60  0001 C CNN
-F 2 "ferris:SW_PG1350" H 7450 1200 60  0001 C CNN
+F 2 "switches:Choc_PG1350_MX_Spacing" H 7450 1200 60  0001 C CNN
 F 3 "" H 7450 1200 60  0000 C CNN
 	1    7450 1200
@@
 F 0 "K1_5" H 7450 2033 60  0000 C CNN
 F 1 "KEYSW" H 7450 1700 60  0001 C CNN
-F 2 "ferris:SW_PG1350" H 7450 1800 60  0001 C CNN
+F 2 "switches:Choc_PG1350_MX_Spacing" H 7450 1800 60  0001 C CNN
 F 3 "" H 7450 1800 60  0000 C CNN
 	1    7450 1800
@@
 F 0 "K1_6" H 8150 2033 60  0000 C CNN
 F 1 "KEYSW" H 8150 1700 60  0001 C CNN
-F 2 "ferris:SW_PG1350" H 8150 1800 60  0001 C CNN
+F 2 "switches:Choc_PG1350_MX_Spacing" H 8150 1800 60  0001 C CNN
 F 3 "" H 8150 1800 60  0000 C CNN
 	1    8150 1800
@@
 F 0 "K0_7" H 8850 1433 60  0000 C CNN
 F 1 "KEYSW" H 8850 1100 60  0001 C CNN
-F 2 "ferris:SW_PG1350" H 8850 1200 60  0001 C CNN
+F 2 "switches:Choc_PG1350_MX_Spacing" H 8850 1200 60  0001 C CNN
 F 3 "" H 8850 1200 60  0000 C CNN
 	1    8850 1200
@@
 F 0 "K0_6" H 8150 1433 60  0000 C CNN
 F 1 "KEYSW" H 8150 1100 60  0001 C CNN
-F 2 "ferris:SW_PG1350" H 8150 1200 60  0001 C CNN
+F 2 "switches:Choc_PG1350_MX_Spacing" H 8150 1200 60  0001 C CNN
 F 3 "" H 8150 1200 60  0000 C CNN
 	1    8150 1200
@@
 F 0 "K1_7" H 8850 2033 60  0000 C CNN
 F 1 "KEYSW" H 8850 1700 60  0001 C CNN
-F 2 "ferris:SW_PG1350" H 8850 1800 60  0001 C CNN
+F 2 "switches:Choc_PG1350_MX_Spacing" H 8850 1800 60  0001 C CNN
 F 3 "" H 8850 1800 60  0000 C CNN
 	1    8850 1800
@@
 F 0 "K2_5" H 7450 2633 60  0000 C CNN
 F 1 "KEYSW" H 7450 2300 60  0001 C CNN
-F 2 "ferris:SW_PG1350" H 7450 2400 60  0001 C CNN
+F 2 "switches:Choc_PG1350_MX_Spacing" H 7450 2400 60  0001 C CNN
 F 3 "" H 7450 2400 60  0000 C CNN
 	1    7450 2400
@@
 F 0 "K2_6" H 8150 2633 60  0000 C CNN
 F 1 "KEYSW" H 8150 2300 60  0001 C CNN
-F 2 "ferris:SW_PG1350" H 8150 2400 60  0001 C CNN
+F 2 "switches:Choc_PG1350_MX_Spacing" H 8150 2400 60  0001 C CNN
 F 3 "" H 8150 2400 60  0000 C CNN
 	1    8150 2400
@@
 F 0 "K2_7" H 8850 2633 60  0000 C CNN
 F 1 "KEYSW" H 8850 2300 60  0001 C CNN
-F 2 "ferris:SW_PG1350" H 8850 2400 60  0001 C CNN
+F 2 "switches:Choc_PG1350_MX_Spacing" H 8850 2400 60  0001 C CNN
 F 3 "" H 8850 2400 60  0000 C CNN
 	1    8850 2400
@@
 F 0 "K0_8" H 9550 1433 60  0000 C CNN
 F 1 "KEYSW" H 9550 1100 60  0001 C CNN
-F 2 "ferris:SW_PG1350" H 9550 1200 60  0001 C CNN
+F 2 "switches:Choc_PG1350_MX_Spacing" H 9550 1200 60  0001 C CNN
 F 3 "" H 9550 1200 60  0000 C CNN
 	1    9550 1200
@@
 F 0 "K1_8" H 9550 2033 60  0000 C CNN
 F 1 "KEYSW" H 9550 1700 60  0001 C CNN
-F 2 "ferris:SW_PG1350" H 9550 1800 60  0001 C CNN
+F 2 "switches:Choc_PG1350_MX_Spacing" H 9550 1800 60  0001 C CNN
 F 3 "" H 9550 1800 60  0000 C CNN
 	1    9550 1800
@@
 F 0 "K2_8" H 9550 2633 60  0000 C CNN
 F 1 "KEYSW" H 9550 2300 60  0001 C CNN
-F 2 "ferris:SW_PG1350" H 9550 2400 60  0001 C CNN
+F 2 "switches:Choc_PG1350_MX_Spacing" H 9550 2400 60  0001 C CNN
 F 3 "" H 9550 2400 60  0000 C CNN
 	1    9550 2400
@@
 F 0 "K0_9" H 10250 1433 60  0000 C CNN
 F 1 "KEYSW" H 10250 1100 60  0001 C CNN
-F 2 "ferris:SW_PG1350" H 10250 1200 60  0001 C CNN
+F 2 "switches:Choc_PG1350_MX_Spacing" H 10250 1200 60  0001 C CNN
 F 3 "" H 10250 1200 60  0000 C CNN
 	1    10250 1200
@@
 F 0 "K1_9" H 10250 2033 60  0000 C CNN
 F 1 "KEYSW" H 10250 1700 60  0001 C CNN
-F 2 "ferris:SW_PG1350" H 10250 1800 60  0001 C CNN
+F 2 "switches:Choc_PG1350_MX_Spacing" H 10250 1800 60  0001 C CNN
 F 3 "" H 10250 1800 60  0000 C CNN
 	1    10250 1800
@@
 F 0 "K2_9" H 10250 2633 60  0000 C CNN
 F 1 "KEYSW" H 10250 2300 60  0001 C CNN
-F 2 "ferris:SW_PG1350" H 10250 2400 60  0001 C CNN
+F 2 "switches:Choc_PG1350_MX_Spacing" H 10250 2400 60  0001 C CNN
 F 3 "" H 10250 2400 60  0000 C CNN
 	1    10250 2400
@@
 F 0 "K3_5" H 7450 3233 60  0000 C CNN
 F 1 "KEYSW" H 7450 2900 60  0001 C CNN
-F 2 "ferris:SW_PG1350" H 7450 3000 60  0001 C CNN
+F 2 "switches:Choc_PG1350_MX_Spacing" H 7450 3000 60  0001 C CNN
 F 3 "" H 7450 3000 60  0000 C CNN
 	1    7450 3000
@@
 F 0 "K3_6" H 8150 3233 60  0000 C CNN
 F 1 "KEYSW" H 8150 2900 60  0001 C CNN
-F 2 "ferris:SW_PG1350" H 8150 3000 60  0001 C CNN
+F 2 "switches:Choc_PG1350_MX_Spacing" H 8150 3000 60  0001 C CNN
 F 3 "" H 8150 3000 60  0000 C CNN
 	1    8150 3000

Commit message: 0.1/base: edit fields and generate netlist to improve bom quality
Parts:
- C2: LCSC Part # (none) -> C1804
- C4, C5, C6: LCSC Part # (none) -> C49678
- D0_1, D0_2, D0_3, D0_4, D0_5, D0_6, D0_7, D0_8, D0_9, D1_0, D1_1, D1_2, D1_3, D1_4, D1_5, D1_6, D1_7, D1_8, D1_9, D2_0, D2_1, D2_2, D2_3, D2_4, D2_5, D2_6, D2_7, D2_8, D2_9, D3_3, D3_4, D3_5, D3_6: LCSC Part # (none) -> C81598
- Jack1: LCSC Part # (none) -> C12569
- K0_0: DNP (none) -> true; LCSC Part # C489144 -> (none)
- K0_1, K0_2, K0_3, K0_4, K0_5, K0_6, K0_7, K0_8, K0_9, K1_0, K1_1, K1_2, K1_3, K1_4, K1_5, K1_6, K1_7, K1_8, K1_9, K2_0, K2_1, K2_2, K2_3, K2_4, K2_5, K2_6, K2_7, K2_8, K2_9, K3_3, K3_4, K3_5, K3_6: DNP (none) -> true
- R2, R9: LCSC Part # (none) -> C17414
- R4: LCSC Part # (none) -> C17561
- R6: LCSC Part # (none) -> C27834
- R8: LCSC Part # (none) -> C17673

Commit message: bom: generate jlc boms too
We had to slightly alter the schematics to match the plugin's
expectations. Adapted the interactive plugin to account for the change.
Parts:
- C1, C2: LCSC Part (none) -> C1804; LCSC Part # C1804 -> (none)
- C10, C3, C4, C5, C6, C9: LCSC Part (none) -> C49678; LCSC Part # C49678 -> (none)
- C7: LCSC Part (none) -> C1779; LCSC Part # C1779 -> (none)
- C8: LCSC Part (none) -> C28323; LCSC Part # C28323 -> (none)
- D0_0, D0_1, D0_2, D0_3, D0_4, D0_5, D0_6, D0_7, D0_8, D0_9, D1_0, D1_1, D1_2, D1_3, D1_4, D1_5, D1_6, D1_7, D1_8, D1_9, D2_0, D2_1, D2_2, D2_3, D2_4, D2_5, D2_6, D2_7, D2_8, D2_9, D3_3, D3_4, D3_5, D3_6: LCSC Part (none) -> C81598; LCSC Part # C81598 -> (none)
- F1: LCSC Part (none) -> C151162; LCSC Part # C151162 -> (none)
- J1: LCSC Part (none) -> C165948; LCSC Part # C165948 -> (none)
- Jack0, Jack1: LCSC Part (none) -> C12569; LCSC Part # C12569 -> (none)
- K0_0, K0_1, K0_2, K0_3, K0_4, K0_5, K0_6, K0_7, K0_8, K0_9, K1_0, K1_1, K1_2, K1_3, K1_4, K1_5, K1_6, K1_7, K1_8, K1_9, K2_0, K2_1, K2_2, K2_3, K2_4, K2_5, K2_6, K2_7, K2_8, K2_9, K3_3, K3_4, K3_5, K3_6: JLCPCB BOM (none) -> false
- R1, R2, R9: LCSC Part (none) -> C17414; LCSC Part # C17414 -> (none)
- R3, R4: LCSC Part (none) -> C17561; LCSC Part # C17561 -> (none)
- R5, R6: LCSC Part (none) -> C27834; LCSC Part # C27834 -> (none)
- R7, R8: LCSC Part (none) -> C17673; LCSC Part # C17673 -> (none)
- SW1: LCSC Part (none) -> C231329; LCSC Part # C231329 -> (none)
- U1: LCSC Part (none) -> C44854; LCSC Part # C44854 -> (none)
- U2: LCSC Part (none) -> C47023; LCSC Part # C47023 -> (none)
- Y1: LCSC Part (none) -> C13738; LCSC Part # C13738 -> (none)
