File: 0.1/high/ferris.kicad_pcb (KiCad board)
At the start: 2 copper layers, 219.1 x 95.2 mm, 102 parts, among them J1 USB C, K0_0 KEYSW, K0_1 KEYSW, K0_2 KEYSW, K0_3 KEYSW, K0_4 KEYSW, K0_5 KEYSW, K0_6 KEYSW, K0_7 KEYSW, K0_8 KEYSW, K0_9 KEYSW, K1_0 KEYSW, K1_1 KEYSW, K1_2 KEYSW, K1_3 KEYSW, K1_4 KEYSW, K1_5 KEYSW, K1_6 KEYSW, K1_7 KEYSW, K1_8 KEYSW, K1_9 KEYSW, K2_0 KEYSW, K2_1 KEYSW, K2_2 KEYSW, K2_3 KEYSW, K2_4 KEYSW, K2_5 KEYSW, K2_6 KEYSW, K2_7 KEYSW, K2_8 KEYSW, K2_9 KEYSW, K3_3 KEYSW, K3_4 KEYSW, K3_5 KEYSW, K3_6 KEYSW, SW1 SW_PUSH, U1 ATmega32U4-AU, U2 MCP23017_SO, Y1 Crystal

Commit message: 0.1/high: update symbols, rerun traces for DRC
Parts:
- G***: footprint ferris:ferris_silk_closed_eyes -> silkscreens:closed_eyes
- G***: footprint ferris:ferris_silk_open_eyes -> silkscreens:open_eyes
- G*** (x2): footprint ferris:tall_ferris_copper_pad -> copper_pads:ferris_high
- K0_0, K0_1, K0_2, K0_3, K0_4, K0_5, K0_6, K0_7, K0_8, K0_9, K1_0, K1_1, K1_2, K1_3, K1_4, K1_5, K1_6, K1_7, K1_8, K1_9, K2_0, K2_1, K2_2, K2_3, K2_4, K2_5, K2_6, K2_7, K2_8, K2_9, K3_3, K3_4, K3_5, K3_6: footprint MX:MXOnly-1U-NoLED -> switches:MX
- Y1: footprint Crystal:Crystal_SMD_3225-4Pin_3.2x2.5mm_HandSoldering -> Crystal:Crystal_SMD_3225-4Pin_3.2x2.5mm
Routing:
- net /row0,0: track 203.5 -> 216.0 mm
- net /col4: track 119.0 -> 107.6 mm
- net /col0: track 95.0 -> 89.7 mm
- net /col9: track 137.6 -> 142.0 mm
- net /col3: track 88.9 -> 87.7 mm
- net /col6: track 94.4 -> 95.3 mm
